Commit message: add image observation to non-hierarchical envs

File: pybullet_multigoal_gym/assets/objects/table.urdf (robot description, URDF)
Before this commit: robot table, 1 links, 0 joints
Links:
- link table: geometry collision box size=0.5 0.7 0.16; visual box size=0.5 0.7 0.16

File: pybullet_multigoal_gym/assets/objects/target.urdf (robot description, URDF)
Before this commit: robot block_target, 1 links, 0 joints
Links:
- link block_target: geometry visual sphere radius=0.02
