Commit message: setup package

File: pybullet_multigoal_gym/assets/objects/block.urdf (robot description, URDF)
Before this commit: robot blue_block, 1 links, 0 joints
Links:
- removed link blue_block
- added link block, mass 0.1; collision box size=0.03 0.03 0.03; visual box size=0.03 0.03 0.03

File: pybullet_multigoal_gym/assets/objects/long_table.urdf (robot description, URDF)
Before this commit: robot red_block, 1 links, 0 joints
Links:
- removed link red_block
- added link table, mass 0; collision box size=1.2 0.5 0.16; visual box size=1.2 0.5 0.16

File: pybullet_multigoal_gym/assets/objects/table.urdf (robot description, URDF)
Before this commit: robot table, 1 links, 0 joints
Links:
- link table: geometry collision box size=0.4 0.4 0.16; visual box size=0.4 0.6 0.16

Commit message: finished parallel jaw env

File: pybullet_multigoal_gym/assets/objects/block.urdf (robot description, URDF)
Before this commit: robot block, 1 links, 0 joints
Links:
- added link iiwa_mocap_link_1, mass 0.0; visual box size=1.0 0.005 0.005
- added link iiwa_mocap_link_2, mass 0.0; visual box size=0.005 1.0 0.005
Joints:
- added joint x_axis: type fixed, parent block, child iiwa_mocap_link_1, origin xyz=0.0 0.0 0.0 rpy=0.0 0.0 0.0
- added joint y_axis: type fixed, parent block, child iiwa_mocap_link_2, origin xyz=0.0 0.0 0.0 rpy=0.0 0.0 0.0

File: pybullet_multigoal_gym/assets/robots/kuka/iiwa14_parallel_jaw.urdf (robot description, URDF)
Before this commit: robot iiwa14, 17 links, 16 joints
Links:
- removed link iiwa_gripper_left_finger
- removed link iiwa_gripper_right_finger
- added link iiwa_gripper_finger1, mass 0.636951; collision box size=0.025, 0.01, 0.08; visual box size=0.025, 0.01, 0.08
- added link iiwa_gripper_finger2, mass 0.636951; collision box size=0.025, 0.01, 0.08; visual box size=0.025, 0.01, 0.08
Joints:
- removed joint iiwa_gripper_left_finger_joint
- removed joint iiwa_gripper_right_finger_joint
- added joint iiwa_gripper_finger1_joint: type prismatic, parent iiwa_gripper_base_link, child iiwa_gripper_finger1, origin xyz=0 0.03 0.04 rpy=0 0 0, axis 0 -1 0, limit lower=0.0 upper=0.025 effort=20 velocity=0.2
- added joint iiwa_gripper_finger2_joint: type prismatic, parent iiwa_gripper_base_link, child iiwa_gripper_finger2, origin xyz=0 -0.03 0.04 rpy=0 0 0, axis 0 1 0, limit lower=0.0 upper=0.025 effort=20 velocity=0.2
- joint iiwa_gripper_finger1_finger_tab_joint: origin xyz=0.0 0.0 0.0 rpy=0.0 0.0 0.0 -> xyz=0.0 -0.005 0.0 rpy=0.0 0.0 0.0; parent iiwa_gripper_left_finger -> iiwa_gripper_finger1
- joint iiwa_gripper_finger2_finger_tab_joint: origin xyz=0.0 0.0 0.0 rpy=0.0 0.0 0.0 -> xyz=0.0 0.005 0.0 rpy=0.0 0.0 0.0; parent iiwa_gripper_right_finger -> iiwa_gripper_finger2
