Commit message: update object mass; add a cylinder bulk to slide env

File: pybullet_multigoal_gym/assets/objects/cylinder_bulk.urdf (robot description, URDF)
Before this commit: robot block, 1 links, 0 joints
Links:
- link block: geometry collision cylinder length=0.02 radius=0.03; visual cylinder length=0.02 radius=0.03
