Commit message: update slide task configuration

File: pybullet_multigoal_gym/assets/objects/long_table.urdf (robot description, URDF)
Before this commit: robot table, 1 links, 0 joints
Links:
- link table: geometry collision box size=1.4 0.7 0.16; visual box size=1.4 0.7 0.16

Commit message: slide task setup

File: pybullet_multigoal_gym/assets/objects/long_table.urdf (robot description, URDF)
Before this commit: robot table, 1 links, 0 joints
Links:
- link table: geometry collision box size=1.0 0.9 0.16; visual box size=1.0 0.9 0.16
