Commit message: chest push $ pick-place tasks

File: pybullet_multigoal_gym/assets/objects/chest_front_sliding_door.urdf (robot description, URDF)
Before this commit: robot chest, 7 links, 6 joints
Links:
- removed link chest_door_bearing
- removed link chest_front_wall
- added link chest_door_handle_keypoint, mass 0.0; visual sphere radius=0.005
- added link chest_door_left_keypoint, mass 0.0; visual sphere radius=0.005
- added link chest_door_right_keypoint, mass 0.0; visual sphere radius=0.005
- added link chest_up_wall, mass 2; collision box size=0.11 0.14 0.01; visual box size=0.11 0.14 0.01
- link chest_door: mass 2 -> 0; geometry collision box size=0.01 0.14 0.10; visual box size=0.01 0.14 0.10
- link chest_door_handle: geometry collision cylinder length=0.04 radius=0.005; visual cylinder length=0.04 radius=0.005
Joints:
- removed joint chest_back_front_wall_joint
- removed joint chest_back_wall_bearing_joint
- removed joint chest_door_bearing_joint
- added joint chest_back_up_wall_joint: type fixed, parent chest_back_wall, child chest_up_wall, origin xyz=0.05 0.0 0.056 rpy=0 0 0
- added joint chest_back_wall_door_joint: type prismatic, parent chest_back_wall, child chest_door, origin xyz=0.10 0.0 0 rpy=0 0 0, axis 0 1 0, limit lower=-0.12 upper=0.12 effort=200 velocity=10
- added joint chest_door_handle_keypoint_joint: type fixed, parent chest_door_handle, child chest_door_handle_keypoint, origin xyz=0.0 0.0 0.02 rpy=0 0 0
- added joint chest_door_left_keypoint_joint: type fixed, parent chest_door, child chest_door_left_keypoint, origin xyz=0.0 -0.07 0.0 rpy=0 0 0
- added joint chest_door_right_keypoint_joint: type fixed, parent chest_door, child chest_door_right_keypoint, origin xyz=0.0 0.07 0.0 rpy=0 0 0
- joint chest_door_handle_joint: origin xyz=0.085    0.0 0.0 rpy=0 1.57 0 -> xyz=0.025 0.0 0.045 rpy=0 1.57 0

Commit message: update chest task curriculum

File: pybullet_multigoal_gym/assets/objects/chest_front_sliding_door.urdf (robot description, URDF)
Before this commit: robot chest, 9 links, 8 joints
Joints:
- joint chest_back_wall_door_joint: limit lower=-0.12 upper=0.12 effort=200 velocity=10 -> lower=0 upper=0.12 effort=200 velocity=1

File: pybullet_multigoal_gym/assets/objects/target_chest.urdf (robot description, URDF)
Before this commit: robot block_target, 1 links, 0 joints
Links:
- link block_target: geometry visual sphere radius=0.05

Commit message: create a stopper on the chest sliding door

File: pybullet_multigoal_gym/assets/objects/chest_front_sliding_door.urdf (robot description, URDF)
Before this commit: robot chest, 9 links, 8 joints
Links:
- added link chest_door_stopper, mass 0; collision box size=0.01 0.14 0.10; visual box size=0.02 0.003 0.003
Joints:
- added joint chest_door_stopper_joint: type fixed, parent chest_door, child chest_door_stopper, origin xyz=-0.006 -0.065 0 rpy=0 0 0
- joint chest_back_wall_door_joint: origin xyz=0.10 0.0 0 rpy=0 0 0 -> xyz=0.105 0.0 0.0 rpy=0 0 0
- joint chest_door_handle_joint: origin xyz=0.025 0.0 0.045 rpy=0 1.57 0 -> xyz=0.025 0.0 0.04 rpy=0 1.57 0

Commit message: some tinkering

File: pybullet_multigoal_gym/assets/objects/chest_front_sliding_door.urdf (robot description, URDF)
Before this commit: robot chest, 10 links, 9 joints
Links:
- removed link chest_door_stopper
- link chest_door_handle: geometry collision cylinder length=0.02 radius=0.005; visual cylinder length=0.02 radius=0.005
Joints:
- removed joint chest_door_stopper_joint
- joint chest_back_wall_door_joint: origin xyz=0.105 0.0 0.0 rpy=0 0 0 -> xyz=0.103 0.0 0.0 rpy=0 0 0
- joint chest_door_handle_joint: origin xyz=0.025 0.0 0.04 rpy=0 1.57 0 -> xyz=0.01 0.0 0.04 rpy=0 1.57 0
- joint chest_door_handle_keypoint_joint: origin xyz=0.0 0.0 0.02 rpy=0 0 0 -> xyz=0.0 0.0 0.01 rpy=0 0 0

Commit message: chest push task modification

File: pybullet_multigoal_gym/assets/objects/chest_front_sliding_door.urdf (robot description, URDF)
Before this commit: robot chest, 9 links, 8 joints
Links:
- removed link chest_up_wall
Joints:
- removed joint chest_back_up_wall_joint
