Commit message: finished arm & gripper motion capture control codes

File: pybullet_multigoal_gym/assets/robots/kuka/iiwa14_robotiq85.urdf (robot description, URDF)
Before this commit: robot iiwa14, 20 links, 19 joints
Links:
- removed link block_0
- removed link table
- added link iiwa_gripper_tip, mass 0.0
Joints:
- removed joint table_block_0_joint
- removed joint world_table_joint
- added joint iiwa_gripper_tip_joint: type fixed, parent iiwa_link_7, child iiwa_gripper_tip, origin xyz=0.0 0.0 0.18 rpy=0.0 0.0 0.0
- joint iiwa_gripper_finger1_finger_tip_joint: limit lower=-3.14 upper=3.14 effort=0.1 velocity=100.0 -> lower=-0.804 upper=0.804 effort=1000 velocity=2.0; mimic joint=iiwa_gripper_finger1_joint multiplier=-1 -> (none)
- joint iiwa_gripper_finger1_inner_knuckle_joint: limit lower=-3.14 upper=3.14 effort=0.1 velocity=100.0 -> lower=0.0 upper=0.804 effort=1000 velocity=2.0; mimic joint=iiwa_gripper_finger1_joint offset=0 -> (none)
- joint iiwa_gripper_finger2_finger_tip_joint: limit lower=-3.14 upper=3.14 effort=0.1 velocity=100.0 -> lower=-0.804 upper=0.804 effort=1000 velocity=2.0; mimic joint=iiwa_gripper_finger1_joint multiplier=-1 -> (none)
- joint iiwa_gripper_finger2_inner_knuckle_joint: limit lower=-3.14 upper=3.14 effort=0.1 velocity=100.0 -> lower=0.0 upper=0.804 effort=1000 velocity=2.0; mimic joint=iiwa_gripper_finger1_joint offset=0 -> (none)
- joint iiwa_gripper_finger2_joint: limit lower=-3.14 upper=3.14 effort=1000 velocity=100.0 -> lower=0.0 upper=0.804 effort=1000 velocity=2.0; mimic joint=iiwa_gripper_finger1_joint -> (none)

Commit message: code structure overhaul

File: pybullet_multigoal_gym/assets/robots/kuka/iiwa14_robotiq85.urdf (robot description, URDF)
Before this commit: robot iiwa14, 19 links, 18 joints
Links:
- removed link world
- added link iiwa_gripper_finger1_finger_tab_link, mass 0.0; visual box size=0.005 0.005 0.005
- added link iiwa_gripper_finger2_finger_tab_link, mass 0.0; visual box size=0.005 0.005 0.005
- added link plane, mass .0; collision box size=10 10 0.002; visual box size=10 10 0.002
- link iiwa_gripper_finger1_finger_link: geometry collision mesh filename=meshes/robotiq_2f_85/collision/robotiq_85_finger_link_new.s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; visual mesh filename=meshes/robotiq_2f_85/visual/robotiq_85_finger_link.dae
- link iiwa_gripper_finger2_finger_link: geometry collision mesh filename=meshes/robotiq_2f_85/collision/robotiq_85_finger_link_new.s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; visual mesh filename=meshes/robotiq_2f_85/visual/robotiq_85_finger_link.dae
- link iiwa_gripper_tip: geometry visual box size=0.005 0.005 0.005
Joints:
- removed joint world_iiwa_joint
- added joint iiwa_gripper_finger1_finger_tab_joint: type fixed, parent iiwa_gripper_finger1_finger_tip_link, child iiwa_gripper_finger1_finger_tab_link, origin xyz=0.05 0.0075 0.0 rpy=0.0 0.0 0.0
- added joint iiwa_gripper_finger2_finger_tab_joint: type fixed, parent iiwa_gripper_finger2_finger_tip_link, child iiwa_gripper_finger2_finger_tab_link, origin xyz=0.05 0.0075 0.0 rpy=0.0 0.0 0.0
- added joint plane_iiwa_joint: type fixed, parent plane, child iiwa_link_0, origin xyz=0 0 0 rpy=0 0 0
- joint iiwa_gripper_finger1_finger_tip_joint: mimic (none) -> joint=iiwa_gripper_finger1_joint multiplier=-1
- joint iiwa_gripper_finger1_inner_knuckle_joint: mimic (none) -> joint=iiwa_gripper_finger1_joint offset=0
- joint iiwa_gripper_finger2_finger_tip_joint: mimic (none) -> joint=iiwa_gripper_finger1_joint multiplier=-1
- joint iiwa_gripper_finger2_inner_knuckle_joint: mimic (none) -> joint=iiwa_gripper_finger1_joint offset=0
- joint iiwa_gripper_tip_joint: origin xyz=0.0 0.0 0.18 rpy=0.0 0.0 0.0 -> xyz=0.0 0.0 0.2 rpy=0.0 0.0 0.0

Commit message: finished the basic framework & implemented the first task, ready to train

File: pybullet_multigoal_gym/assets/robots/kuka/iiwa14_robotiq85.urdf (robot description, URDF)
Before this commit: robot iiwa14, 21 links, 20 joints
Links:
- link plane: geometry collision box size=5 5 0.002; visual box size=5 5 0.002
Joints:
- joint iiwa_gripper_tip_joint: origin xyz=0.0 0.0 0.2 rpy=0.0 0.0 0.0 -> xyz=0.0 0.0 0.18 rpy=0.0 0.0 0.0

Commit message: bugs; adjust obj poses

File: pybullet_multigoal_gym/assets/robots/kuka/iiwa14_robotiq85.urdf (robot description, URDF)
Before this commit: robot iiwa14, 21 links, 20 joints
Links:
- added link iiwa_mocap_link_1, mass 0.0; visual box size=1.0 0.005 0.005
- added link iiwa_mocap_link_2, mass 0.0; visual box size=0.005 1.0 0.005
Joints:
- added joint iiwa_gripper_mocap_joint1: type fixed, parent iiwa_gripper_tip, child iiwa_mocap_link_1, origin xyz=0.0 0.0 0.0 rpy=0.0 0.0 0.0
- added joint iiwa_gripper_mocap_joint2: type fixed, parent iiwa_gripper_tip, child iiwa_mocap_link_2, origin xyz=0.0 0.0 0.0 rpy=0.0 0.0 0.0
