Commit message: finished parallel jaw urdf tests

File: pybullet_multigoal_gym/assets/robots/kuka/iiwa14_parallel_jaw.urdf (robot description, URDF)
Before this commit: robot iiwa14, 23 links, 22 joints
Links:
- removed link iiwa_gripper_finger1_finger_link
- removed link iiwa_gripper_finger1_finger_tip_link
- removed link iiwa_gripper_finger1_inner_knuckle_link
- removed link iiwa_gripper_finger1_knuckle_link
- removed link iiwa_gripper_finger2_finger_link
- removed link iiwa_gripper_finger2_finger_tip_link
- removed link iiwa_gripper_finger2_inner_knuckle_link
- removed link iiwa_gripper_finger2_knuckle_link
- added link iiwa_gripper_left_finger, mass 0.636951; collision box size=0.025, 0.01, 0.08; visual box size=0.025, 0.01, 0.08
- added link iiwa_gripper_right_finger, mass 0.636951; collision box size=0.025, 0.01, 0.08; visual box size=0.025, 0.01, 0.08
- link iiwa_gripper_base_link: geometry collision cylinder length=0.04 radius=0.05; visual cylinder length=0.04 radius=0.05
Joints:
- removed joint iiwa_gripper_finger1_finger_joint
- removed joint iiwa_gripper_finger1_finger_tip_joint
- removed joint iiwa_gripper_finger1_inner_knuckle_joint
- removed joint iiwa_gripper_finger1_joint
- removed joint iiwa_gripper_finger2_finger_joint
- removed joint iiwa_gripper_finger2_finger_tip_joint
- removed joint iiwa_gripper_finger2_inner_knuckle_joint
- removed joint iiwa_gripper_finger2_joint
- added joint iiwa_gripper_left_finger_joint: type prismatic, parent iiwa_gripper_base_link, child iiwa_gripper_left_finger, origin xyz=0 0.03 0.04 rpy=0 0 0, axis 0 -1 0, limit lower=0.0 upper=0.02 effort=20 velocity=0.2
- added joint iiwa_gripper_right_finger_joint: type prismatic, parent iiwa_gripper_base_link, child iiwa_gripper_right_finger, origin xyz=0 -0.03 0.04 rpy=0 0 0, axis 0 1 0, limit lower=0.0 upper=0.02 effort=20 velocity=0.2
- joint iiwa_gripper_base_joint: origin xyz=0 0 0.045 rpy=0 -1.57079632679 0 -> xyz=0 0 0.055 rpy=0 0 0
- joint iiwa_gripper_finger1_finger_tab_joint: origin xyz=0.05 0.0075 0.0 rpy=0.0 0.0 0.0 -> xyz=0.0 0.0 0.0 rpy=0.0 0.0 0.0; parent iiwa_gripper_finger1_finger_tip_link -> iiwa_gripper_left_finger
- joint iiwa_gripper_finger2_finger_tab_joint: origin xyz=0.05 0.0075 0.0 rpy=0.0 0.0 0.0 -> xyz=0.0 0.0 0.0 rpy=0.0 0.0 0.0; parent iiwa_gripper_finger2_finger_tip_link -> iiwa_gripper_right_finger
- joint iiwa_gripper_tip_joint: origin xyz=0.0 0.0 0.18 rpy=0.0 0.0 0.0 -> xyz=0.0 0.0 0.12 rpy=0.0 0.0 0.0

Commit message: debug parallel jaw & ik

File: pybullet_multigoal_gym/assets/robots/kuka/iiwa14_parallel_jaw.urdf (robot description, URDF)
Before this commit: robot iiwa14, 17 links, 16 joints
Joints:
- joint iiwa_gripper_finger1_joint: limit lower=0.0 upper=0.025 effort=20 velocity=0.2 -> lower=0.0 upper=0.03 effort=20 velocity=0.2; origin xyz=0 0.03 0.04 rpy=0 0 0 -> xyz=0 0.04 0.04 rpy=0 0 0
- joint iiwa_gripper_finger2_joint: limit lower=0.0 upper=0.025 effort=20 velocity=0.2 -> lower=0.0 upper=0.03 effort=20 velocity=0.2; origin xyz=0 -0.03 0.04 rpy=0 0 0 -> xyz=0 -0.04 0.04 rpy=0 0 0

Commit message: gripper bug

File: pybullet_multigoal_gym/assets/robots/kuka/iiwa14_parallel_jaw.urdf (robot description, URDF)
Before this commit: robot iiwa14, 17 links, 16 joints
Joints:
- joint iiwa_gripper_finger1_joint: limit lower=0.0 upper=0.03 effort=20 velocity=0.2 -> lower=0.0 upper=0.035 effort=20 velocity=0.2
- joint iiwa_gripper_finger2_joint: limit lower=0.0 upper=0.03 effort=20 velocity=0.2 -> lower=0.0 upper=0.035 effort=20 velocity=0.2

Commit message: on-hand camera observation support

File: pybullet_multigoal_gym/assets/robots/kuka/iiwa14_parallel_jaw.urdf (robot description, URDF)
Before this commit: robot iiwa14, 17 links, 16 joints
Links:
- added link iiwa_hand_cam_origin, mass 0.0; visual box size=0.01 0.01 0.01
Joints:
- added joint iiwa_hand_cam_joint: type fixed, parent iiwa_link_7, child iiwa_hand_cam_origin, origin xyz=0.22 0.0 -0.1 rpy=0.0 0.0 0.0

File: pybullet_multigoal_gym/assets/robots/kuka/iiwa14_robotiq85.urdf (robot description, URDF)
Before this commit: robot iiwa14, 23 links, 22 joints
Links:
- added link iiwa_hand_cam_origin, mass 0.0; visual box size=0.01 0.01 0.01
Joints:
- added joint iiwa_hand_cam_joint: type fixed, parent iiwa_link_7, child iiwa_hand_cam_origin, origin xyz=0.22 0.0 -0.1 rpy=0.0 0.0 0.0

Commit message: cam settings

File: pybullet_multigoal_gym/assets/robots/kuka/iiwa14_parallel_jaw.urdf (robot description, URDF)
Before this commit: robot iiwa14, 18 links, 17 joints
Joints:
- joint iiwa_hand_cam_joint: origin xyz=0.22 0.0 -0.1 rpy=0.0 0.0 0.0 -> xyz=0.2 0.0 0.0 rpy=0.0 0.0 0.0
