Commit message: add 0 mass initial

File: pybullet_multigoal_gym/assets/objects/assembling_shape/slot.urdf (robot description, URDF)
Before this commit: robot slot, 4 links, 3 joints
Links:
- link slot_target: mass None -> 0

File: pybullet_multigoal_gym/assets/objects/assembling_shape/workspace.urdf (robot description, URDF)
Before this commit: robot workspace, 2 links, 1 joints
Links:
- link range: mass None -> 0
