Commit message: primitive push task; transparent object target

File: pybullet_multigoal_gym/assets/objects/assembling_shape/cube_target.urdf (robot description, URDF)
Before this commit: robot block_target, 1 links, 0 joints
Links:
- removed link block_target
- added link cube_target, mass 0; visual box size=0.03 0.03 0.03

File: pybullet_multigoal_gym/assets/objects/assembling_shape/slot_target.urdf (robot description, URDF)
Before this commit: robot slot, 4 links, 3 joints
Links:
- link base: mass 100 -> 0; geometry visual box size=0.03 0.09 0.03
- link left: mass 100 -> 0; geometry visual box size=0.03 0.03 0.03
- link right: mass 100 -> 0; geometry visual box size=0.03 0.03 0.03
